File: BLDC_V_0.1/MCU_STM32.kicad_sch (KiCad schematic)
At the start: 31 parts, among them J2 SWD, J3 Conn_01x03, J5 USB_B_Micro, U3 AMS1117, U3 USBLC6-2SC6, U5 STM32G473VET6, Y1 24MHz

Commit message: Schematic prototip done.
Parts:
- C10, C12, C15, C16, C4, C5, C6, C7, C8, C9: footprint (none) -> Capacitor_SMD:C_0402_1005Metric
- C11, C16, C17: footprint (none) -> Capacitor_SMD:C_0603_1608Metric
- L2: footprint 15EDGVC:CONN_15EDGVC-3.5-03P-1X_DEG -> Inductor_SMD:L_0603_1608Metric
- R8: footprint (none) -> Resistor_SMD:R_0402_1005Metric
- U5: footprint STM32G473VET6:LQFP100-14x14mm -> LQFP100-14x14mm
Changed lines of the file:
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@@
       (effects (font (size 1.27 1.27)) (justify left))
     )
-    (property "Footprint" "" (at 279.0952 36.576 0)
+    (property "Footprint" "Capacitor_SMD:C_0603_1608Metric" (at 279.0952 36.576 0)
       (effects (font (size 1.27 1.27)) hide)
     )
@@
       (effects (font (size 1.524 1.524)) (justify left))
     )
-    (property "Footprint" "STM32G473VET6:LQFP100-14x14mm" (at 149.225 29.21 0)
+    (property "Footprint" "LQFP100-14x14mm" (at 149.225 29.21 0)
       (effects (font (size 1.27 1.27) italic) hide)
     )
@@
       (effects (font (size 1.27 1.27)) (justify left))
     )
-    (property "Footprint" "" (at 31.75 189.738 0)
+    (property "Footprint" "Capacitor_SMD:C_0402_1005Metric" (at 31.75 189.738 0)
       (effects (font (size 1.27 1.27)) hide)
     )
@@
       (effects (font (size 1.27 1.27)) (justify left))
     )
-    (property "Footprint" "" (at 233.3752 36.576 0)
+    (property "Footprint" "Capacitor_SMD:C_0402_1005Metric" (at 233.3752 36.576 0)
       (effects (font (size 1.27 1.27)) hide)
     )
@@
       (effects (font (size 1.27 1.27)) hide)
     )
-    (property "Datasheet" "" (at 234.95 108.585 0)
+    (property "Datasheet" "https://www.st.com/resource/en/datasheet/usblc6-2.pdf" (at 234.95 108.585 0)
       (effects (font (size 1.27 1.27)) hide)
     )
@@
       (effects (font (size 1.27 1.27)))
     )
-    (property "Footprint" "15EDGVC:CONN_15EDGVC-3.5-03P-1X_DEG" (at 244.221 53.975 0)
+    (property "Footprint" "Inductor_SMD:L_0603_1608Metric" (at 244.221 53.975 0)
       (effects (font (size 1.27 1.27)) hide)
     )
@@
       (effects (font (size 1.27 1.27)) (justify left))
     )
-    (property "Footprint" "" (at 210.5152 36.576 0)
+    (property "Footprint" "Capacitor_SMD:C_0402_1005Metric" (at 210.5152 36.576 0)
       (effects (font (size 1.27 1.27)) hide)
     )
@@
       (effects (font (size 1.27 1.27)) (justify left))
     )
-    (property "Footprint" "" (at 221.9452 36.576 0)
+    (property "Footprint" "Capacitor_SMD:C_0402_1005Metric" (at 221.9452 36.576 0)
       (effects (font (size 1.27 1.27)) hide)
     )
@@
       (effects (font (size 1.27 1.27)) (justify left))
     )
-    (property "Footprint" "" (at 266.3952 36.576 0)
+    (property "Footprint" "Capacitor_SMD:C_0402_1005Metric" (at 266.3952 36.576 0)
       (effects (font (size 1.27 1.27)) hide)
     )
@@
       (effects (font (size 1.27 1.27)) (justify left))
     )
-    (property "Footprint" "" (at 19.05 189.738 0)
+    (property "Footprint" "Capacitor_SMD:C_0402_1005Metric" (at 19.05 189.738 0)
       (effects (font (size 1.27 1.27)) hide)
     )
@@
       (effects (font (size 1.27 1.27)) (justify left))
     )
-    (property "Footprint" "" (at 188.2902 64.135 0)
+    (property "Footprint" "Capacitor_SMD:C_0603_1608Metric" (at 188.2902 64.135 0)
       (effects (font (size 1.27 1.27)) hide)
     )
@@
       (effects (font (size 1.27 1.27)) (justify left))
     )
-    (property "Footprint" "" (at 31.75 176.403 0)
+    (property "Footprint" "Resistor_SMD:R_0402_1005Metric" (at 31.75 176.403 0)
       (effects (font (size 1.27 1.27)) hide)
     )
@@
       (effects (font (size 1.27 1.27)) (justify left))
     )
-    (property "Footprint" "" (at 225.1202 64.135 0)
+    (property "Footprint" "Capacitor_SMD:C_0603_1608Metric" (at 225.1202 64.135 0)
       (effects (font (size 1.27 1.27)) hide)
     )
@@
       (effects (font (size 1.27 1.27)) (justify left))
     )
-    (property "Footprint" "" (at 258.826 57.15 0)
+    (property "Footprint" "Capacitor_SMD:C_0402_1005Metric" (at 258.826 57.15 0)
       (effects (font (size 1.27 1.27)) hide)
     )
@@
       (effects (font (size 1.27 1.27)) (justify left))
     )
-    (property "Footprint" "" (at 254.9652 36.576 0)
+    (property "Footprint" "Capacitor_SMD:C_0402_1005Metric" (at 254.9652 36.576 0)
       (effects (font (size 1.27 1.27)) hide)
     )
@@
       (effects (font (size 1.27 1.27)) (justify left))
     )
-    (property "Footprint" "" (at 202.8952 85.725 0)
+    (property "Footprint" "Capacitor_SMD:C_0402_1005Metric" (at 202.8952 85.725 0)
       (effects (font (size 1.27 1.27)) hide)
     )
@@
       (effects (font (size 1.27 1.27)) (justify left))
     )
-    (property "Footprint" "" (at 215.5952 85.725 0)
+    (property "Footprint" "Capacitor_SMD:C_0603_1608Metric" (at 215.5952 85.725 0)
       (effects (font (size 1.27 1.27)) hide)
     )
@@
     )
   )
-  (symbol (lib_name "STM32G473VET6_1") (lib_id "STM32G473:STM32G473VET6") (at 33.02 30.48 0) (unit 1)
+  (symbol (lib_id "STM32G473:STM32G473VET6") (at 33.02 30.48 0) (unit 1)
     (in_bom yes) (on_board yes) (dnp no)
     (property "Reference" "U5" (at 51.054 24.384 0)
@@
       (effects (font (size 1.524 1.524)) (justify left))
     )
-    (property "Footprint" "STM32G473VET6:LQFP100-14x14mm" (at 33.02 30.48 0)
+    (property "Footprint" "LQFP100-14x14mm" (at 33.02 30.48 0)
       (effects (font (size 1.27 1.27) italic) hide)
     )
@@
       (effects (font (size 1.27 1.27)) (justify left))
     )
-    (property "Footprint" "" (at 199.0852 36.576 0)
+    (property "Footprint" "Capacitor_SMD:C_0402_1005Metric" (at 199.0852 36.576 0)
       (effects (font (size 1.27 1.27)) hide)
     )
@@
       (effects (font (size 1.27 1.27)) (justify left))
     )
-    (property "Footprint" "" (at 249.555 57.785 0)
+    (property "Footprint" "Capacitor_SMD:C_0603_1608Metric" (at 249.555 57.785 0)
       (effects (font (size 1.27 1.27)) hide)
     )
@@
       (effects (font (size 1.27 1.27)) (justify left))
     )
-    (property "Footprint" "" (at 243.5352 36.576 0)
-      (effects (font (size 1.27 1.27)) hide)
-    )
+    (property "Footprint" "Capacitor_SMD:C_0402_1005Metric" (at 243.5352 36.576 0)
+      (effects (font (size 1.27 1.27)) hide)
+    )

Commit message: PCB placement completed.
Parts:
- J3: footprint Connector:FanPinHeader_1x03_P2.54mm_Vertical -> Connector_PinHeader_2.54mm:PinHeader_1x03_P2.54mm_Vertical
- U5: footprint LQFP100-14x14mm -> STM32G473VET6:LQFP100-14x14mm
Connections:
- net DRV_CS: now also U5.51 (PB12); no longer U5.26 (PA4)
- net DRV_ENABLE: now also U5.62 (PD15); no longer U5.8 (PC14-OSC32_IN)
- net EXT_SPI_CS: now also U5.26 (PA4); no longer U5.51 (PB12)
- net EXT_SPI_MISO: now also U5.28 (PA6); no longer U5.53 (PB14)
- net EXT_SPI_MOSI: now also U5.29 (PA7); no longer U5.54 (PB15)
- net EXT_SPI_SCK: now also U5.27 (PA5); no longer U5.52 (PB13)
- net HALL_A: now also U5.56 (PD9); no longer U5.21 (PA1)
- net HALL_B: now also U5.55 (PD8); no longer U5.22 (PA2)
- net HALL_C: now also U5.50 (PB11); no longer U5.25 (PA3)
- net SPI_MISO: now also U5.53 (PB14); no longer U5.28 (PA6)
- net SPI_MOSI: now also U5.54 (PB15); no longer U5.29 (PA7)
- net SPI_SCK: now also U5.52 (PB13); no longer U5.27 (PA5)
- net TEMP_IN: now also U5.47 (PB10); no longer U5.20 (PA0)
